File: Kicad/Riegamatico_MQTT/Riegamatico_MQTT.sch (KiCad schematic (older format))
At the start: 11 parts, among them J1 LCD I2C, J10 SENS TEMP TIERRA, J2 CONTROL CARGA, J3 BATERIA 12V, J5 BOMBA, J6 SENS NIVEL, J7 SENS CAUDAL, J8 SENS AMBIENTE, J9 SENS HUMEDAD TIERRA, Q1 FET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

Commit message: Up
Parts:
- added J0: POWER 5V, symbol Connector_Generic:Conn_01x02
Connections:
- net +5V: now also J0.1 (Pin_1)
- net GND: now also J0.2 (Pin_2)
Other:
- note added: "RIEGAMATICO MQTT\nDiego Maroto - BilbaoMakers\nGNU General Public License v3.0"
Changed lines of the file:
@@
 L power:+5V #PWR?
 U 1 1 5D1383EB
-P 2400 1100
-F 0 "#PWR?" H 2400 950 50  0001 C CNN
-F 1 "+5V" H 2415 1273 50  0000 C CNN
-F 2 "" H 2400 1100 50  0001 C CNN
-F 3 "" H 2400 1100 50  0001 C CNN
-	1    2400 1100
+P 2400 750
+F 0 "#PWR?" H 2400 600 50  0001 C CNN
+F 1 "+5V" H 2415 923 50  0000 C CNN
+F 2 "" H 2400 750 50  0001 C CNN
+F 3 "" H 2400 750 50  0001 C CNN
+	1    2400 750
 	1    0    0    -1
 $EndComp
@@
 	2400 4200 4500 4200
 Wire Wire Line
-	2400 1100 2400 4200
+	2400 750  2400 4200
 $Comp
 L power:GND #PWR?
@@
 L power:+3V3 #PWR?
 U 1 1 5D138991
-P 2800 1100
-F 0 "#PWR?" H 2800 950 50  0001 C CNN
-F 1 "+3V3" H 2815 1273 50  0000 C CNN
-F 2 "" H 2800 1100 50  0001 C CNN
-F 3 "" H 2800 1100 50  0001 C CNN
-	1    2800 1100
-	1    0    0    -1
-$EndComp
-Wire Wire Line
-	2800 1100 2800 2400
+P 2800 750
+F 0 "#PWR?" H 2800 600 50  0001 C CNN
+F 1 "+3V3" H 2815 923 50  0000 C CNN
+F 2 "" H 2800 750 50  0001 C CNN
+F 3 "" H 2800 750 50  0001 C CNN
+	1    2800 750
+	1    0    0    -1
+$EndComp
+Wire Wire Line
+	2800 750  2800 2400
 Wire Wire Line
 	2800 2400 4500 2400
 Wire Wire Line
-	9700 750  9700 900
-Wire Wire Line
-	9700 900  9850 900
+	9350 750  9350 900
+Wire Wire Line
+	9350 900  9850 900
 Wire Wire Line
 	9850 1000 7350 1000
@@
 L power:+5V #PWR?
 U 1 1 5D138DDF
-P 9700 750
-F 0 "#PWR?" H 9700 600 50  0001 C CNN
-F 1 "+5V" H 9715 923 50  0000 C CNN
-F 2 "" H 9700 750 50  0001 C CNN
-F 3 "" H 9700 750 50  0001 C CNN
-	1    9700 750
+P 9350 750
+F 0 "#PWR?" H 9350 600 50  0001 C CNN
+F 1 "+5V" H 9365 923 50  0000 C CNN
+F 2 "" H 9350 750 50  0001 C CNN
+F 3 "" H 9350 750 50  0001 C CNN
+	1    9350 750
 	1    0    0    -1
 $EndComp
@@
 Wire Wire Line
 	9350 1700 9350 900
-Wire Wire Line
-	9350 900  9700 900
-Connection ~ 9700 900
+Connection ~ 9350 900
 Wire Wire Line
 	9850 2100 9500 2100
@@
 Connection ~ 9500 4800
 Wire Wire Line
-	9500 4800 9500 5900
+	9500 4800 9500 5450
 Wire Wire Line
 	9850 3900 8350 3900
@@
 Wire Wire Line
 	6450 3200 6450 4200
+$Comp
+L Connector_Generic:Conn_01x02 J0
+U 1 1 5D173D7E
+P 10050 5350
+F 0 "J0" H 10130 5342 50  0000 L CNN
+F 1 "POWER 5V" H 10130 5251 50  0000 L CNN
+F 2 "" H 10050 5350 50  0001 C CNN
+F 3 "~" H 10050 5350 50  0001 C CNN
+	1    10050 5350
+	1    0    0    -1
+$EndComp
+Wire Wire Line
+	9850 5450 9500 5450
+Connection ~ 9500 5450
+Wire Wire Line
+	9500 5450 9500 5900
+$Comp
+L power:+5V #PWR?
+U 1 1 5D1760AC
+P 9650 5250
+F 0 "#PWR?" H 9650 5100 50  0001 C CNN
+F 1 "+5V" H 9665 5423 50  0000 C CNN
+F 2 "" H 9650 5250 50  0001 C CNN
+F 3 "" H 9650 5250 50  0001 C CNN
+	1    9650 5250
+	1    0    0    -1
+$EndComp
+Wire Wire Line
+	9650 5250 9650 5350
+Wire Wire Line
+	9650 5350 9850 5350
+Text Notes 7100 6950 0    50   ~ 10
+RIEGAMATICO MQTT\nDiego Maroto - BilbaoMakers\nGNU General Public License v3.0
 $EndSCHEMATC
